File: pcb/CameraBoard.sch (KiCad schematic (older format))
At the start: 12 parts

Commit message: PCB with FIFO
Parts:
- removed U? (x2): shiftregister_74HC595, symbol shiftregister_74HC595
- added C?: 1uF, symbol C
- added FIFO? (x2): fifo_74HC40105, symbol fifo_74HC40105
- added P?: CONN_01X05, symbol CONN_01X05
- added SH?: shiftregister_74HC165, symbol shiftregister_74HC165
- added SH?: shiftregister_74HC595, symbol shiftregister_74HC595
- added U? (x2): notgate_74HCT04, symbol notgate_74HCT04
Connections:
- net +5V: now also C?.1, FIFO?.16 (VCC), FIFO?.16 (VCC), SH?.10 (SRCLR), SH?.16 (VCC), SH?.16 (VCC), U?.14 (VCC)
- net GND: now also C?.2, FIFO?.1 (~OE), FIFO?.1 (~OE), FIFO?.8 (GND), FIFO?.8 (GND), FIFO?.9 (Reset), FIFO?.9 (Reset), SH?.10 (serial_in), SH?.13 (~OE), SH?.8 (GND), SH?.8 (GND), U?.7 (GND)
- net Arduino_SPI_Clock: now reaches LS?.5 (2A), U?.1 ((led)(SCK)D13)
- net Arduino_SPI_Clock: now also SH?.11 (SRCLK)
- net Arduinio_SPI_Data: now reaches LS?.7 (3A), U?.29 ((MOSI)#D11)
- net Arduinio_SPI_Data: now also SH?.14 (SER)
- net Pixel_D7: no longer names the net of OV7670?.9 (D7)
- net Pixel_D7: no longer U?.25 (D7)
- new net: P?.2 (P2), SH?.1 (~Parallel_load), U?.3
- new net: FIFO?.13 (Q0), SH?.11 (D0)
- new net: FIFO?.12 (Q1), SH?.12 (D1)
- new net: FIFO?.11 (Q2), SH?.13 (D2)
- new net: FIFO?.10 (Q3), SH?.14 (D3)
- new net: P?.3 (P3), SH?.15 (~Clock_enable)
- new net: P?.4 (P4), SH?.2 (Clock)
- new net: FIFO?.13 (Q0), SH?.3 (D4)
- new net: FIFO?.12 (Q1), SH?.4 (D5)
- new net: FIFO?.11 (Q2), SH?.5 (D6)
- new net: FIFO?.10 (Q3), SH?.6 (D7)
- new net: P?.5 (P5), SH?.9 (Q7)
- new net: FIFO?.14 (DOR), P?.1 (P1)
- new net: FIFO?.15 (~Shift_out), FIFO?.15 (~Shift_out), U?.4
- new net: FIFO?.3 (Shift_in), FIFO?.3 (Shift_in), U?.2
- new net: FIFO?.4 (D0), SH?.15 (Q0)
- new net: FIFO?.5 (D1), SH?.1 (Q1)
- new net: FIFO?.6 (D2), SH?.2 (Q2)
- new net: FIFO?.7 (D3), SH?.3 (Q3)
- new net: FIFO?.4 (D0), SH?.4 (Q4)
- new net: FIFO?.5 (D1), SH?.5 (Q5)
- new net: FIFO?.6 (D2), SH?.6 (Q6)
- new net: FIFO?.7 (D3), SH?.7 (Q7)
- new net Arduino_P7: SH?.12 (RCLK), U?.1, U?.25 (D7)
- no-connect marks 6 -> 12
Other:
- moved on the sheet: C?, LS?, TFT?

Commit message: PCB footprints are not set
Parts:
- removed P?: CONN_01X02, symbol CONN_01X02
- removed P?: CONN_01X05, symbol CONN_01X05
- added P4: CONN_01X08, Pin_Headers:Pin_Header_Straight_2x04, symbol CONN_01X08
- added PWR1: power_connection, Pin_Headers:Pin_Header_Straight_1x02, symbol power_connection
- C1, C2: renamed from C?; footprint (none) -> Capacitors_SMD:C_1206_HandSoldering
- FIFO1, FIFO2: renamed from FIFO?; footprint (none) -> Housings_SOIC:SOIC-16_3.9x9.9mm_Pitch1.27mm
- LS1: renamed from LS?; footprint (none) -> Housings_SOIC:SOIC-16_3.9x9.9mm_Pitch1.27mm
- OV76701: renamed from OV7670?; footprint (none) -> Pin_Headers:Pin_Header_Straight_2x09
- P2, P3: renamed from P?; footprint (none) -> Pin_Headers:Pin_Header_Straight_1x03
- R1, R2: renamed from R?; footprint (none) -> Resistors_SMD:R_1206_HandSoldering
- SH1, SH2: renamed from SH?; footprint (none) -> Housings_SOIC:SOIC-16_3.9x9.9mm_Pitch1.27mm
- TFT1: renamed from TFT?; footprint (none) -> Pin_Headers:Pin_Header_Straight_2x04
- U1: renamed from U?; footprint DIL20 -> arduino:arduino_mini
- U2: renamed from U?; footprint (none) -> Housings_SOIC:SOIC-16_3.9x9.9mm_Pitch1.27mm
Connections:
- net +5V: now also PWR1.1 (VCC)
- net Arduino_P7: now also U2.3; no longer U2.1
- net GND: now also PWR1.2 (GND)
- net at SH1.1 (~Parallel_load): now also U2.1, P4.2 (P2); no longer U2.3
- net at SH1.15 (~Clock_enable): now also P4.3 (P3)
- net at SH1.2 (Clock): now also P4.4 (P4)
- net at SH1.9 (Q7): now also P4.5 (P5)
- net at FIFO1.14 (DOR): now also P4.1 (P1)
- net at FIFO1.15 (~Shift_out), FIFO2.15 (~Shift_out): now also U2.2; no longer U2.4
- net at FIFO1.3 (Shift_in), FIFO2.3 (Shift_in): now also U2.4; no longer U2.2
- no-connect marks 12 -> 16
