File: pcb/CameraBoard.sch (KiCad schematic (older format))
At the start: 17 parts, among them P2 CONN_01X03, P3 CONN_01X03, P4 CONN_01X08, U1 arduino_mini, U2 notgate_74HCT04

Commit message: Fixed NOT gate footprint
Parts:
- U2: footprint Housings_SOIC:SOIC-16_3.9x9.9mm_Pitch1.27mm -> Housings_SOIC:SOIC-14_3.9x8.7mm_Pitch1.27mm
Changed lines of the file:
@@
 F 0 "U2" H 3850 5950 50  0000 C CNN
 F 1 "notgate_74HCT04" H 4100 5750 50  0000 C CNN
-F 2 "Housings_SOIC:SOIC-16_3.9x9.9mm_Pitch1.27mm" H 3700 5850 50  0001 C CNN
+F 2 "Housings_SOIC:SOIC-14_3.9x8.7mm_Pitch1.27mm" H 3700 5850 50  0001 C CNN
 F 3 "" H 3700 5850 50  0000 C CNN
 	2    3700 5850
@@
 F 0 "U2" H 6850 4600 50  0000 C CNN
 F 1 "notgate_74HCT04" H 6900 4300 50  0000 C CNN
-F 2 "Housings_SOIC:SOIC-16_3.9x9.9mm_Pitch1.27mm" H 6700 4500 50  0001 C CNN
+F 2 "Housings_SOIC:SOIC-14_3.9x8.7mm_Pitch1.27mm" H 6700 4500 50  0001 C CNN
 F 3 "" H 6700 4500 50  0000 C CNN
 	1    6700 4500
@@
 $EndComp
 $Comp
-L GND #PWR?
+L GND #PWR031
 U 1 1 5738DE02
 P 9450 5950
-F 0 "#PWR?" H 9450 5700 50  0001 C CNN
+F 0 "#PWR031" H 9450 5700 50  0001 C CNN
 F 1 "GND" H 9450 5800 50  0000 C CNN
 F 2 "" H 9450 5950 50  0000 C CNN
