File: pcb/CameraBoard.kicad_pcb (KiCad board)
At the start: 2 copper layers, 17 parts, among them P2 CONN_01X03, P3 CONN_01X03, P4 CONN_01X08, U1 arduino_mini, U2 notgate_74HCT04

Commit message: Fixed NOT gate footprint
Parts:
- U2: footprint Housings_SOIC:SOIC-16_3.9x9.9mm_Pitch1.27mm -> Housings_SOIC:SOIC-14_3.9x8.7mm_Pitch1.27mm
- moved U2 0.64 mm to (148.1, 125.7)
Other:
- board text added: "Indrek Luuk"
- board text added: "v1.1"
Changed lines of the file:
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@@
     (area 130.718167 84.545951 180.413 132.788001)
     (thickness 1.6)
-    (drawings 0)
-    (tracks 635)
+    (drawings 2)
+    (tracks 636)
     (zones 0)
     (modules 17)
@@
     (visible_elements 7FFEFFFF)
     (pcbplotparams
-      (layerselection 0x000f0_80000001)
+      (layerselection 0x010f0_80000001)
       (usegerberextensions true)
       (excludeedgelayer true)
@@
       (net 44 "Net-(OV76701-Pad7)"))
   )
-  (module Housings_SOIC:SOIC-16_3.9x9.9mm_Pitch1.27mm (layer B.Cu)
-    (at 148.209 125.095)
-    (descr "16-Lead Plastic Small Outline (SL) - Narrow, 3.90 mm Body [SOIC] (see Microchip Packaging Specification 00000049BS.pdf)")
-    (tags "SOIC 1.27")
-    (attr smd)
-    (fp_text reference U2 (at 0 6) (layer B.SilkS)
-      (effects (font (size 1 1) (thickness 0.15)) (justify mirror))
-    )
-    (fp_text value notgate_74HCT04 (at 0 -6) (layer B.Fab)
-      (effects (font (size 1 1) (thickness 0.15)) (justify mirror))
-    )
-    (fp_line (start -3.7 5.25) (end -3.7 -5.25) (layer B.CrtYd) (width 0.05))
-    (fp_line (start 3.7 5.25) (end 3.7 -5.25) (layer B.CrtYd) (width 0.05))
-    (fp_line (start -3.7 5.25) (end 3.7 5.25) (layer B.CrtYd) (width 0.05))
-    (fp_line (start -3.7 -5.25) (end 3.7 -5.25) (layer B.CrtYd) (width 0.05))
-    (fp_line (start -2.075 5.075) (end -2.075 4.97) (layer B.SilkS) (width 0.15))
-    (fp_line (start 2.075 5.075) (end 2.075 4.97) (layer B.SilkS) (width 0.15))
-    (fp_line (start 2.075 -5.075) (end 2.075 -4.97) (layer B.SilkS) (width 0.15))
-    (fp_line (start -2.075 -5.075) (end -2.075 -4.97) (layer B.SilkS) (width 0.15))
-    (fp_line (start -2.075 5.075) (end 2.075 5.075) (layer B.SilkS) (width 0.15))
-    (fp_line (start -2.075 -5.075) (end 2.075 -5.075) (layer B.SilkS) (width 0.15))
-    (fp_line (start -2.075 4.97) (end -3.45 4.97) (layer B.SilkS) (width 0.15))
-    (pad 1 smd rect (at -2.7 4.445) (size 1.5 0.6) (layers B.Cu B.Paste B.Mask)
-      (net 55 "Net-(P4-Pad2)"))
-    (pad 2 smd rect (at -2.7 3.175) (size 1.5 0.6) (layers B.Cu B.Paste B.Mask)
-      (net 15 "Net-(FIFO1-Pad15)"))
-    (pad 3 smd rect (at -2.7 1.905) (size 1.5 0.6) (layers B.Cu B.Paste B.Mask)
-      (net 63 Arduino_P7))
-    (pad 4 smd rect (at -2.7 0.635) (size 1.5 0.6) (layers B.Cu B.Paste B.Mask)
-      (net 5 "Net-(FIFO1-Pad3)"))
-    (pad 5 smd rect (at -2.7 -0.635) (size 1.5 0.6) (layers B.Cu B.Paste B.Mask))
-    (pad 6 smd rect (at -2.7 -1.905) (size 1.5 0.6) (layers B.Cu B.Paste B.Mask))
-    (pad 7 smd rect (at -2.7 -3.175) (size 1.5 0.6) (layers B.Cu B.Paste B.Mask)
-      (net 1 GND))
-    (pad 8 smd rect (at -2.7 -4.445) (size 1.5 0.6) (layers B.Cu B.Paste B.Mask))
-    (pad 9 smd rect (at 2.7 -4.445) (size 1.5 0.6) (layers B.Cu B.Paste B.Mask))
-    (pad 10 smd rect (at 2.7 -3.175) (size 1.5 0.6) (layers B.Cu B.Paste B.Mask))
-    (pad 11 smd rect (at 2.7 -1.905) (size 1.5 0.6) (layers B.Cu B.Paste B.Mask))
-    (pad 12 smd rect (at 2.7 -0.635) (size 1.5 0.6) (layers B.Cu B.Paste B.Mask))
-    (pad 13 smd rect (at 2.7 0.635) (size 1.5 0.6) (layers B.Cu B.Paste B.Mask))
-    (pad 14 smd rect (at 2.7 1.905) (size 1.5 0.6) (layers B.Cu B.Paste B.Mask)
-      (net 3 +5V))
-    (pad 15 smd rect (at 2.7 3.175) (size 1.5 0.6) (layers B.Cu B.Paste B.Mask))
-    (pad 16 smd rect (at 2.7 4.445) (size 1.5 0.6) (layers B.Cu B.Paste B.Mask))
-    (model Housings_SOIC.3dshapes/SOIC-16_3.9x9.9mm_Pitch1.27mm.wrl
-      (at (xyz 0 0 0))
-      (scale (xyz 1 1 1))
-      (rotate (xyz 0 0 0))
-    )
-  )
   (module Pin_Headers:Pin_Header_Straight_1x02 (layer F.Cu)
     (at 153.7335 91.44 90)
@@
       (rotate (xyz 0 0 90))
     )
+  )
+  (module Housings_SOIC:SOIC-14_3.9x8.7mm_Pitch1.27mm (layer B.Cu)
+    (at 148.1455 125.73)
+    (descr "14-Lead Plastic Small Outline (SL) - Narrow, 3.90 mm Body [SOIC] (see Microchip Packaging Specification 00000049BS.pdf)")
+    (tags "SOIC 1.27")
+    (attr smd)
+    (fp_text reference U2 (at 0 5.375) (layer B.SilkS)
+      (effects (font (size 1 1) (thickness 0.15)) (justify mirror))
+    )
+    (fp_text value notgate_74HCT04 (at 0 -5.375) (layer B.Fab)
+      (effects (font (size 1 1) (thickness 0.15)) (justify mirror))
+    )
+    (fp_line (start -3.7 4.65) (end -3.7 -4.65) (layer B.CrtYd) (width 0.05))
+    (fp_line (start 3.7 4.65) (end 3.7 -4.65) (layer B.CrtYd) (width 0.05))
+    (fp_line (start -3.7 4.65) (end 3.7 4.65) (layer B.CrtYd) (width 0.05))
+    (fp_line (start -3.7 -4.65) (end 3.7 -4.65) (layer B.CrtYd) (width 0.05))
+    (fp_line (start -2.075 4.45) (end -2.075 4.335) (layer B.SilkS) (width 0.15))
+    (fp_line (start 2.075 4.45) (end 2.075 4.335) (layer B.SilkS) (width 0.15))
+    (fp_line (start 2.075 -4.45) (end 2.075 -4.335) (layer B.SilkS) (width 0.15))
+    (fp_line (start -2.075 -4.45) (end -2.075 -4.335) (layer B.SilkS) (width 0.15))
+    (fp_line (start -2.075 4.45) (end 2.075 4.45) (layer B.SilkS) (width 0.15))
+    (fp_line (start -2.075 -4.45) (end 2.075 -4.45) (layer B.SilkS) (width 0.15))
+    (fp_line (start -2.075 4.335) (end -3.45 4.335) (layer B.SilkS) (width 0.15))
+    (pad 1 smd rect (at -2.7 3.81) (size 1.5 0.6) (layers B.Cu B.Paste B.Mask)
+      (net 55 "Net-(P4-Pad2)"))
+    (pad 2 smd rect (at -2.7 2.54) (size 1.5 0.6) (layers B.Cu B.Paste B.Mask)
+      (net 15 "Net-(FIFO1-Pad15)"))
+    (pad 3 smd rect (at -2.7 1.27) (size 1.5 0.6) (layers B.Cu B.Paste B.Mask)
+      (net 63 Arduino_P7))
+    (pad 4 smd rect (at -2.7 0) (size 1.5 0.6) (layers B.Cu B.Paste B.Mask)
+      (net 5 "Net-(FIFO1-Pad3)"))
+    (pad 5 smd rect (at -2.7 -1.27) (size 1.5 0.6) (layers B.Cu B.Paste B.Mask))
+    (pad 6 smd rect (at -2.7 -2.54) (size 1.5 0.6) (layers B.Cu B.Paste B.Mask))
+    (pad 7 smd rect (at -2.7 -3.81) (size 1.5 0.6) (layers B.Cu B.Paste B.Mask)
+      (net 1 GND))
+    (pad 8 smd rect (at 2.7 -3.81) (size 1.5 0.6) (layers B.Cu B.Paste B.Mask))
+    (pad 9 smd rect (at 2.7 -2.54) (size 1.5 0.6) (layers B.Cu B.Paste B.Mask))
+    (pad 10 smd rect (at 2.7 -1.27) (size 1.5 0.6) (layers B.Cu B.Paste B.Mask))
+    (pad 11 smd rect (at 2.7 0) (size 1.5 0.6) (layers B.Cu B.Paste B.Mask))
+    (pad 12 smd rect (at 2.7 1.27) (size 1.5 0.6) (layers B.Cu B.Paste B.Mask))
+    (pad 13 smd rect (at 2.7 2.54) (size 1.5 0.6) (layers B.Cu B.Paste B.Mask))
+    (pad 14 smd rect (at 2.7 3.81) (size 1.5 0.6) (layers B.Cu B.Paste B.Mask)
+      (net 3 +5V))
+    (model Housings_SOIC.3dshapes/SOIC-14_3.9x8.7mm_Pitch1.27mm.wrl
+      (at (xyz 0 0 0))
+      (scale (xyz 1 1 1))
+      (rotate (xyz 0 0 0))
+    )
+  )
+  (gr_text v1.1 (at 179.0065 129.0955 90) (layer B.SilkS)
+    (effects (font (size 1.5 1.5) (thickness 0.3)) (justify mirror))
+  )
+  (gr_text "Indrek Luuk" (at 179.0065 94.0435 90) (layer B.SilkS)
+    (effects (font (size 1.5 1.5) (thickness 0.3)) (justify mirror))
   )
   (segment (start 137.287 116.967) (end 138.557 116.967) (width 0.25) (layer B.Cu) (net 1))
@@
   (segment (start 162.687 95.5675) (end 163.4805 94.774) (width 0.25) (layer B.Cu) (net 2))
   (via (at 162.687 95.5675) (size 0.6) (drill 0.4) (layers F.Cu B.Cu) (net 2))
+  (segment (start 150.8455 129.54) (end 152.5905 129.54) (width 0.25) (layer B.Cu) (net 3))
+  (segment (start 153.416 128.7145) (end 156.1465 128.7145) (width 0.25) (layer F.Cu) (net 3))
+  (segment (start 152.5905 129.54) (end 153.416 128.7145) (width 0.25) (layer F.Cu) (net 3))
+  (via (at 152.5905 129.54) (size 0.6) (drill 0.4) (layers F.Cu B.Cu) (net 3))
+  (segment (start 156.1465 128.7145) (end 156.21 128.778) (width 0.25) (layer F.Cu) (net 3))
   (segment (start 140.8735 114.6175) (end 139.5095 114.6175) (width 0.25) (layer B.Cu) (net 3))
   (segment (start 139.7 104.267) (end 140.843 105.41) (width 0.25) (layer F.Cu) (net 3))
@@
   (via (at 142.5575 129.4765) (size 0.6) (drill 0.4) (layers F.Cu B.Cu) (net 3))
   (segment (start 142.621 129.4765) (end 142.5575 129.4765) (width 0.25) (layer F.Cu) (net 3))
-  (segment (start 150.909 127) (end 152.5905 127) (width 0.25) (layer B.Cu) (net 3))
-  (segment (start 154.3685 128.778) (end 156.21 128.778) (width 0.25) (layer F.Cu) (net 3))
-  (segment (start 152.5905 127) (end 154.3685 128.778) (width 0.25) (layer F.Cu) (net 3))
-  (via (at 152.5905 127) (size 0.6) (drill 0.4) (layers F.Cu B.Cu) (net 3))
   (segment (start 133.1595 116.2685) (end 133.1595 116.967) (width 0.25) (layer B.Cu) (net 5))
   (segment (start 143.002 125.73) (end 141.605 124.333) (width 0.25) (layer B.Cu) (net 5))
